File: eagle/9doFORK.sch (EAGLE design)
At the start: 39 parts, among them IC1 ATMEGA32U4-MU, SW1 SPST_TACT-KMR2, U2 SPX3819-3.3, U3 MCP73831T-2ACI/OT, X3 microUSB, Y1 32.768kHz, Y2 8MHz

Commit message: fixed some bugs in rawdata-rx, working on rev 2 for board, added expenses info
Parts:
- added R15, R16: 10k, microbuilder:RESISTOR0603MINI
- added X1: TSW-106-02-S-S, con-samtec:TSW-106-02-S-S
- C1, C2: device microbuilder:CAP_CERAMIC0805-NOOUTLINE -> microbuilder:CAP_CERAMIC_0603
- C3: device microbuilder:CAP_CERAMIC0805-NOOUTLINE -> microbuilder:CAP_CERAMIC0603MINI
- C4: device microbuilder:CAP_CERAMIC0805_10MGAP -> microbuilder:CAP_CERAMIC_0603
- C8: device microbuilder:CAP_CERAMIC0603_NO -> microbuilder:CAP_CERAMIC0603MINI
- L: device microbuilder:LED0805_NOOUTLINE -> microbuilder:LED0805
- R1, R11, R12, R13, R14, R2, R6, R7, R8, R9: device microbuilder:RESISTOR_0603_NOOUT -> microbuilder:RESISTOR0603MINI
- R10: device microbuilder:RESISTOR_0603MP -> microbuilder:RESISTOR0603MINI
- R3, R4, R5: device microbuilder:RESISTOR0805_NOOUTLINE -> microbuilder:RESISTOR0603MINI
Connections:
- removed net D4: IC1.PD4(ICP1/ADC8)
- removed net D7: IC1.PE6(INT.6/AIN0)
- new net N$13: JP2.8, R15.2, R16.1
- net A0: now also X1-6.1
- net A1: now also X1-5.1
- net A2: now also X1-4.1
- net A3: now also X1-3.1
- net A4: now also X1-2.1
- net A5: now also X1-1.1
- net CE: now also IC1.PE6(INT.6/AIN0); no longer IC1.PC6(OC3A/!OC4A)
- net CSN: now also IC1.PB0(SS); no longer IC1.PD7(OC4D/ADC10/T0)
- net IRQ: now also R15.1; no longer JP2.8
- net RST: now also R16.2
